File: variants/minimal_32_64B/z80-Arduino_minmal_32B.kicad_sch (KiCad schematic)
At the start: 31 parts, among them SW1 SW_Push, SW3 SW_Push, U1 Z80CPU, U2 74HC373 (74HC573), U3 8282

Commit message: Update version
Parts:
- added R16, R17, R18, R19, R20, R21, R22, R23: 2k2, symbol Device:R
- added U4: 74HC373 (74HC573), symbol 74xx:74HC373
- added U5: KCSA02-107, Display_7Segment:KCSC02-107, symbol Display_Character:KCSA02-107
Connections:
- net A5 (64B) is gone; now on net A5: JP1.3 (B)
- net WR (32B) is gone; now on net IORQ: JP1.1 (A)
- net +5V: now also U4.20 (VCC), U5.3 (CA), U5.8 (CA)
- net D0: now also U4.3 (D0)
- net D1: now also U4.4 (D1)
- net D2: now also U4.7 (D2)
- net D3: now also U4.8 (D3)
- net D4: now also U4.13 (D4)
- net D5: now also U4.14 (D5)
- net D6: now also U4.17 (D6)
- net D7: now also U4.18 (D7)
- net GND: now also U4.10 (GND)
- net IORQ: now also U4.11 (LE); no longer A1.15 (D12)
- net WR: now also A1.21 (A2), U4.1 (OE)
- net at JP1.2 (C): now also A1.15 (D12); no longer A1.21 (A2)
- new net: R21.1, U4.15 (O5)
- new net: R21.2, U5.9 (F)
- new net: R23.1, U4.19 (O7)
- new net: R23.2, U5.5 (DP)
- new net: R19.1, U4.9 (O3)
- new net: R19.2, U5.2 (D)
- new net: R20.1, U4.12 (O4)
- new net: R20.2, U5.1 (E)
- new net: R18.1, U4.6 (O2)
- new net: R18.2, U5.4 (C)
- new net: R22.2, U5.10 (G)
- new net: R17.2, U5.6 (B)
- new net: R16.2, U5.7 (A)
- new net: R22.1, U4.16 (O6)
- new net: R16.1, U4.2 (O0)
- new net: R17.1, U4.5 (O1)
Other:
- note added: "Simple port variation 1 - 7 segment Any OUTPUT port"
- moved on the sheet: JP1

Commit message: Fix 32
Parts:
- removed BZ1, BZ2: Buzzer, symbol Device:Buzzer
- removed D5, D6: LED_RGBK, symbol Device:LED_RGBK
- removed R10, R11, R12, R13, R14, R15, R16, R17, R18, R19, R20, R21, R22, R23: 2k2, symbol Device:R
- removed U4: 74HC373 (74HC573), symbol 74xx:74HC373
- removed U5: KCSA02-107, Display_7Segment:KCSC02-107, symbol Display_Character:KCSA02-107
- added DS?: WC1602A, Display:WC1602A, symbol Display_Character:WC1602A
- added Q?: 2N3904, Package_TO_SOT_THT:TO-92_Inline, symbol Transistor_BJT:2N3904
- added R?: 2k2, symbol Device:R
- added R?: 4k7, symbol Device:R
- added RV?: 20k, symbol Device:R_Potentiometer
Connections:
- net +5V: now also DS?.15 (LED(+)), DS?.2 (VDD), R?.2, RV?.1
- net A0: now also DS?.4 (RS)
- net D0: now also DS?.7 (D0)
- net D1: now also DS?.8 (D1)
- net D2: now also DS?.9 (D2)
- net D3: now also DS?.10 (D3)
- net D4: now also DS?.11 (D4)
- net D5: now also DS?.12 (D5)
- net D6: now also DS?.13 (D6)
- net D7: now also DS?.14 (D7)
- net GND: now also DS?.1 (VSS), DS?.16 (LED(-)), DS?.5 (R/W), Q?.1 (E), RV?.3
- net IORQ: now also R?.1
- net PA7: now reaches U2.19 (O7)
- net PA7: now also U3.12 (O7)
- net PA1: now reaches U2.5 (O1)
- net PA1: now also U3.18 (O1)
- net PA4: now reaches U2.12 (O4)
- net PA4: now also U3.15 (O4)
- net PA5: now reaches U2.15 (O5)
- net PA5: now also U3.14 (O5)
- net PA6: now reaches U2.16 (O6)
- net PA6: now also U3.13 (O6)
- net PA0: now reaches U2.2 (O0)
- net PA0: now also U3.19 (O0)
- net PA2: now reaches U2.6 (O2)
- net PA2: now also U3.17 (O2)
- net PA3: now reaches U2.9 (O3)
- net PA3: now also U3.16 (O3)
- new net: DS?.3 (VO), RV?.2
- new net: DS?.6 (E), Q?.3 (C), R?.1
- new net: Q?.2 (B), R?.2
- no-connect marks 26 -> 18
Other:
- note removed: "Simple port variation 1 - 7 segment Any OUTPUT port"
- moved on the sheet: U2, U3

Commit message: Fix changes before IDDLE
Parts:
- removed Q?: 2N3904, Package_TO_SOT_THT:TO-92_Inline, symbol Transistor_BJT:2N3904
- removed R?: 2k2, symbol Device:R
- removed R?: 4k7, symbol Device:R
- removed U2: 74HC373 (74HC573), symbol 74xx:74HC373
- removed U3: 8282, symbol Custom_components:8282
- added A?: Arduino_Nano_v2.x, Module:Arduino_Nano, symbol MCU_Module:Arduino_Nano_v2.x
- added R10: 4k7, symbol Device:R
- added U2, U? (x2): 74HC14, symbol 74xx:74HC14
- added U3: 74HCT573, symbol 74xx:74HCT574
- added U? (x4): 74LS32, symbol 74xx:74LS32
- added U?: 74HC244, symbol 74xx:74HC244
- gave numbers to parts that had none: 2
Connections:
- net +5V: now also A?.27 (+5V), R10.1, U3.20 (VCC), U?.20 (VCC)
- net A0: now also A?.19 (A0)
- net A1: now also A?.20 (A1)
- net A2: now also A?.21 (A2)
- net CLK: now also R10.2
- net D0: now also A?.11 (D8), U3.2 (D0), U?.18 (1Y0)
- net D1: now also A?.12 (D9), U3.3 (D1), U?.16 (1Y1)
- net D2: now also A?.13 (D10), U3.4 (D2), U?.14 (1Y2)
- net D3: now also A?.14 (D11), U3.5 (D3), U?.12 (1Y3)
- net D4: now also A?.7 (D4), U3.6 (D4), U?.3 (2Y0)
- net D5: now also A?.8 (D5), U3.7 (D5), U?.5 (2Y1)
- net D6: now also A?.9 (D6), U3.8 (D6), U?.7 (2Y2)
- net D7: now also A?.10 (D7), U3.9 (D7), U?.9 (2Y3)
- net GND: now also C1.1, A?.29 (GND), A?.4 (GND), U3.1 (OE), U3.10 (GND), U?.10 (GND); no longer C1.2
- net IORQ: now also A?.5 (D2), U?.10, U?.13
- net PA0: now also U3.19 (Q0)
- net PA1: now also U3.18 (Q1)
- net PA2: now also U3.17 (Q2)
- net PA3: now also U3.16 (Q3)
- net PA4: now also U3.15 (Q4)
- net PA5: now also U3.14 (Q5)
- net PA6: now also U3.13 (Q6)
- net PA7: now also U3.12 (Q7)
- net RD: now also A?.15 (D12), U?.2
- net WR: now also A?.16 (D13), U?.5
- net at DS1.6 (E): now also U2.4
- net at R2.2, SW1.2, U1.26 (~{RESET}): now also C1.2; no longer C1.1
- net A6: now reaches U1.36 (A6)
- net A6: now also U?.13
- net A7: now reaches U1.37 (A7)
- net A7: now also A?.6 (D3), U?.12
- new net: U?.1 (1OE), U?.19 (2OE), U?.4
- new net: U2.2, U3.11 (Cp)
- new net !A6: A?.22 (A3), U?.12, U?.9
- new net Analog: A?.26 (A7)
- new net IORQ_0: U?.1, U?.11, U?.4
- new net IORQ_1: U2.3, U?.8
- new net IO_RD: U?.3, U?.3
- new net IO_WR: U2.1, U?.6
- new net PB0: U?.2 (1A0)
- new net PB1: U?.4 (1A1)
- new net PB2: U?.6 (1A2)
- new net PB3: U?.8 (1A3)
- new net PB4: U?.17 (2A0)
- new net PB5: U?.15 (2A1)
- new net PB6: U?.13 (2A2)
- new net PB7: U?.11 (2A3)
- new net RX_PORT: A?.1 (D1/TX)
- new net Reset: A?.28 (~{RESET}), A?.3 (~{RESET})
- new net SCL: A?.23 (A4)
- new net SDA: A?.24 (A5)
- new net TX_PORT: A?.2 (D0/RX)
- no-connect marks 18 -> 20
Other:
- note added: "(00h ... 0Fh)"
- note added: "(C0h ... FFh)"
- note added: "IO Select"
- note added: "Main Arduino"
- note added: "Simple input port"
- note added: "Simple out port"
- note added: "Simple port action selector"
- note added: "Universal port Arduino 0 - Serial UART 1 - Serial Status 2 - I2C 3 - I2C Status 4 - ADC LSB 5 - ADC MSB 6 - ADC 8bit 7 - Random"
- note added: "Universal port Arduino I2C, UART, Analog, Random"
- note removed: "Simple port variation 1 Any OUTPUT port"
- note removed: "Simple port variation 2 Any OUTPUT port"
- moved on the sheet: A1, C1, D1, D2, D3, D4, DS1, JP1, R2, R3, R4, R5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
